File: LH550WF1-breakout/LH550WF1-breakout.kicad_pcb (KiCad board)
At the start: 2 copper layers, 34.3 x 30.5 mm, 3 parts, among them P1 LH550WF1, P2 CONN_02X10

Commit message: Moved component and module libraries into their own repository
The new repo is at cyrozap/KiCad.
Parts:
- P1: footprint HDMI-to-MIPI:GB042-30S -> connectors:GB042-30S
Changed lines of the file:
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@@
     )
   )
-  (module HDMI-to-MIPI:GB042-30S (layer B.Cu)
+  (module connectors:GB042-30S (layer B.Cu)
     (at 148.59 107.95 90)
     (descr http://www.lsmtron.com/pdf/LS%20Mtron%20Connector.pdf)
