File: SSD2828QN4-breakout/SSD2828QN4-breakout.kicad_pcb (KiCad board)
At the start: 2 copper layers, 18 parts, among them P1 CONN_01X30, P10 CONN_01X02, P11 CONN_01X03, P2 CONN_01X02, P3 CONN_01X05, P4 CONN_01X02, P5 CONN_01X02, P6 CONN_01X03, P7 CONN_02X10, P8 CONN_01X02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

Commit message: Moved component and module libraries into their own repository
The new repo is at cyrozap/KiCad.
Parts:
- P1: footprint HDMI-to-MIPI:TE_3-1734592-0 -> connectors:TE_3-1734592-0
- U1: footprint HDMI-to-MIPI:SSD2828QN4 -> miscellaneous:SSD2828QN4
Changed lines of the file:
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@@
     (add_net "Net-(R3-Pad1)")
   )
-  (module HDMI-to-MIPI:SSD2828QN4 (layer F.Cu)
+  (module miscellaneous:SSD2828QN4 (layer F.Cu)
     (at 168.72 109.83)
     (solder_mask_margin 0.02)
@@
       (net 3 /CLK2))
   )
-  (module HDMI-to-MIPI:TE_3-1734592-0 (layer F.Cu)
+  (module connectors:TE_3-1734592-0 (layer F.Cu)
     (at 194.769 109.444 90)
     (descr http://www.te.com/commerce/DocumentDelivery/DDEController?Action=srchrtrv&DocNm=1734592&DocType=Customer+Drawing&DocLang=English)

Commit message: Updated library and replaced SSD2828QN4 footprint
Parts:
- U1: footprint miscellaneous:SSD2828QN4 -> miscellaneous:QFN-68-1EP_8x8mm_Pitch0.4mm
