File: HDMI-to-LH550WF1/Control.sch (KiCad schematic (older format))
At the start: 48 parts

Commit message: Annotated schematic and associated footprints
Parts:
- C35, C36, C37, C38, C39, C40, C41, C42, C43, C44, C45, C46, C47, C48, C49: renamed from C?; footprint (none) -> Capacitors_SMD:C_0402
- C50: renamed from C?; footprint (none) -> Capacitors_SMD:C_0603
- D10, D11, D12, D13, D14, D6, D7, D8, D9: renamed from D?; footprint (none) -> LEDs:LED_0603
- JP13: renamed from JP?; footprint (none) -> Pin_Headers:Pin_Header_Straight_1x02
- P4: renamed from P?; footprint (none) -> Connect:IDC_Header_Straight_20pins
- P5: renamed from P?; footprint (none) -> Pin_Headers:Pin_Header_Straight_1x03
- R26, R27, R28, R29, R30, R31, R32, R33, R34, R35, R36, R37, R38, R39, R40, R41: renamed from R?; footprint (none) -> Resistors_SMD:R_0402
- U10, U9: renamed from U?; footprint (none) -> miscellaneous:UMLP-12_1.8x1.8mm_Pitch0.4mm
- U11: renamed from U?; footprint LQFP48 -> Housings_QFP:LQFP-48_7x7mm_Pitch0.5mm
- gave numbers to parts that had none: 1
Connections:
- no-connect marks 10 -> 23
