File: HDMI-to-LH550WF1/Control.sch (KiCad schematic (older format))
At the start: 46 parts, among them P4 CONN_02X10, P5 CONN_01X03, U10 FXMA2104UMX, U11 STM32F103C8Tx, U9 FXMA2104UMX, Y1 8MHz

Commit message: Fixed issues with STM32 schematic
- Replaced 20-pin JTAG connector with 10-pin Cortex-M debug connector.
- Added USB resistors.
- Switched from 47k I2C pull-ups to 4.7k.
- Removed all those LEDs.
- Renamed the JTAG and UART nets for clarity.
- Switched to a smaller crystal.
- Used 0402 1uF capacitor in place of 0603 one.
Parts:
- removed D10, D11, D12, D13, D6, D7, D8, D9: Green, LEDs:LED_0603, symbol Led_Small
- removed JP13: Jumper_NO_Small, Pin_Headers:Pin_Header_Straight_1x02, symbol Jumper_NO_Small
- removed P4: CONN_02X10, Connect:IDC_Header_Straight_20pins, symbol CONN_02X10
- removed R30, R33, R34, R35, R36, R37, R38, R39, R40: 1k, Resistors_SMD:R_0402, symbol R_Small
- added J2: CONN_02X05, symbol CONN_02X05
- added R16: 1.5k, Resistors_SMD:R_0402, symbol R_Small
- added R17, R19: 22R, Resistors_SMD:R_0402, symbol R_Small
- C50: footprint Capacitors_SMD:C_0603 -> Capacitors_SMD:C_0402
- R27, R29: value 47k -> 4.7k
- Y1: value 8MHz -> ABM3-8.000MHz-D2Y-T; footprint Crystals:Crystal_HC49-SD_SMD -> Crystals:Crystal_SMD_Abracon_ABM3-2pin_5.0x3.2mm
Connections:
- net labels added: JTAG_TCK, JTAG_TDI, JTAG_TDO, JTAG_TMS, UART_RX, UART_TX
- net labels removed: LED0, LED1, LED2, LED3, LED4, LED5, LED6, LED7, RX, TCK, TDI, TDO, TMS, TX, ~TRST~
- wire segments 150 -> 114
- no-connect marks 24 -> 30
Other:
- note removed: "Crystal is ABLS-8.000MHZ-B4-T."
- moved on the sheet: R27, R28, R29

Commit message: Assigned debug connector footprint
Parts:
- J2: footprint (none) -> connectors:FTSH-105-XX-XXX-DV-XXX
Changed lines of the file:
@@
 F 0 "J2" H 10150 1700 50  0000 C CNN
 F 1 "CONN_02X05" H 10150 1100 50  0000 C CNN
-F 2 "" H 10150 200 50  0001 C CNN
+F 2 "connectors:FTSH-105-XX-XXX-DV-XXX" H 10150 200 50  0001 C CNN
 F 3 "" H 10150 200 50  0001 C CNN
 	1    10150 1400
