File: HDMI-to-LH550WF1/HDMI-Bridge.sch (KiCad schematic (older format))
At the start: 25 parts

Commit message: Annotated schematic and associated footprints
Parts:
- C1, C10, C11, C12, C13, C14, C2, C3, C4, C5, C6, C7, C8, C9: renamed from C?; footprint (none) -> Capacitors_SMD:C_0402
- R1, R2, R3, R4, R5, R6, R7, R8, R9: renamed from R?; footprint (none) -> Resistors_SMD:R_0402
- U1: renamed from U?; footprint VLGA-4_2.5x2.0mm -> miscellaneous:VLGA-4_2.5x2.0mm
- U2: renamed from U?; footprint (none) -> miscellaneous:VFBGA-80_7x7mm_Pitch0.65mm
