File: HDMI-to-LH550WF1/Power.sch (KiCad schematic (older format))
At the start: 51 parts

Commit message: Annotated schematic and associated footprints
Parts:
- C23, C24, C25, C31, C32, C34: renamed from C?; footprint (none) -> Capacitors_SMD:C_0603
- C26, C29, C30: renamed from C?; footprint (none) -> SMD_Packages:SMD-1206_Pol
- C27, C28, C33: renamed from C?; footprint (none) -> Capacitors_SMD:C_0402
- D2, D3, D4, D5: renamed from D?; footprint (none) -> LEDs:LED_0603
- JP1, JP10, JP11, JP12, JP2, JP3, JP4, JP5, JP6, JP7, JP8, JP9: renamed from JP?; footprint (none) -> Pin_Headers:Pin_Header_Straight_1x02
- L3: renamed from L?; footprint (none) -> Resistors_SMD:R_0603
- Q1, Q2, Q3: renamed from Q?; footprint (none) -> TO_SOT_Packages_SMD:SOT-23
- R11, R12, R13, R14, R15, R16, R17, R18, R19, R20, R21, R22, R23, R24, R25: renamed from R?; footprint (none) -> Resistors_SMD:R_0402
- U6, U7, U8: renamed from U?; footprint (none) -> TO_SOT_Packages_SMD:SOT-23-5
- gave numbers to parts that had none: 1

Commit message: Fixed issues with power subsystem
- Removed extra power LEDs.
- Switched to 0402 1uF capacitors.
- Power LED is now 0805 instead of 0603.
- Removed jumpers for current/voltage measurements to save space.
Parts:
- removed C26, C29: 10uF, SMD_Packages:SMD-1206_Pol, symbol CP1_Small
- removed C30: 22uF, SMD_Packages:SMD-1206_Pol, symbol CP1_Small
- removed D3, D4, D5: Led_Small, LEDs:LED_0603, symbol Led_Small
- removed JP1, JP11, JP3, JP4, JP5, JP6: Jumper_NC_Small, Pin_Headers:Pin_Header_Straight_1x02, symbol Jumper_NC_Small
- removed JP10, JP12, JP2, JP7, JP8, JP9: Jumper_NO_Small, Pin_Headers:Pin_Header_Straight_1x02, symbol Jumper_NO_Small
- removed Q1, Q2, Q3: 2N2222, TO_SOT_Packages_SMD:SOT-23, symbol Q_NPN_BEC
- removed R16, R20, R21: 100R, Resistors_SMD:R_0402, symbol R_Small
- removed R17, R22, R23: 100k, Resistors_SMD:R_0402, symbol R_Small
- removed R19, R24, R25: 1k, Resistors_SMD:R_0402, symbol R_Small
- added C26, C29: 10uF, Capacitors_SMD:C_1206, symbol C_Small
- added C30: 22uF, Capacitors_SMD:C_1206, symbol C_Small
- C23, C24, C25: footprint Capacitors_SMD:C_0603 -> Capacitors_SMD:C_0402
- C31, C32, C34: value 1uF/X5R -> 1uF; footprint Capacitors_SMD:C_0603 -> Capacitors_SMD:C_0402
- D2: footprint LEDs:LED_0603 -> LEDs:LED_0805
Connections:
- wire segments 84 -> 42
Other:
- note removed: "Transistors are MMBT2222LT1G."
