File: HDMI-to-LH550WF1/Power.sch (KiCad schematic (older format))
At the start: 24 parts, among them U5 AZ1117H-3.3TRE1, U6 AP2127K-1.8TRG1, U7 AP2127K-1.2TRG1, U8 AP2127K-ADJTRG1

Commit message: Added test points to LCD-Panel and Power sheets
Parts:
- added J10, J11, J12, J13, J7, J8, J9: TEST_1P, symbol TEST_1P
Connections:
- net +1V1: now also J12.1
- net +1V2: now also J11.1
- net +1V8: now also J10.1
- net +3V3: now also J9.1
- net +5V: now also J8.1
- net GND: now also J13.1
- net USB_VBUS: now also J7.1

Commit message: Assigned test point footprints
Parts:
- J10, J11, J12, J7, J8, J9: footprint (none) -> Measurement_Points:Measurement_Point_Round-SMD-Pad_Small
- J13: footprint (none) -> Pin_Headers:Pin_Header_Straight_1x01_Pitch2.54mm
Changed lines of the file:
@@
 $EndDescr
 $Comp
-L +1V1 #PWR66
+L +1V1 #PWR043
 U 1 1 583A2A43
 P 5100 5500
-F 0 "#PWR66" H 5100 5350 50  0001 C CNN
+F 0 "#PWR043" H 5100 5350 50  0001 C CNN
 F 1 "+1V1" H 5100 5640 50  0000 C CNN
 F 2 "" H 5100 5500 50  0000 C CNN
@@
 $EndComp
 $Comp
-L +1V2 #PWR64
+L +1V2 #PWR044
 U 1 1 583A2A57
 P 4300 4500
-F 0 "#PWR64" H 4300 4350 50  0001 C CNN
+F 0 "#PWR044" H 4300 4350 50  0001 C CNN
 F 1 "+1V2" H 4300 4640 50  0000 C CNN
 F 2 "" H 4300 4500 50  0000 C CNN
@@
 $EndComp
 $Comp
-L +1V8 #PWR63
+L +1V8 #PWR045
 U 1 1 583A2A6B
 P 4300 3500
-F 0 "#PWR63" H 4300 3350 50  0001 C CNN
+F 0 "#PWR045" H 4300 3350 50  0001 C CNN
 F 1 "+1V8" H 4300 3640 50  0000 C CNN
 F 2 "" H 4300 3500 50  0000 C CNN
@@
 $EndComp
 $Comp
-L +3V3 #PWR62
+L +3V3 #PWR046
 U 1 1 583A2A7F
 P 4100 2500
-F 0 "#PWR62" H 4100 2350 50  0001 C CNN
+F 0 "#PWR046" H 4100 2350 50  0001 C CNN
 F 1 "+3V3" H 4100 2640 50  0000 C CNN
 F 2 "" H 4100 2500 50  0000 C CNN
@@
 $EndComp
 $Comp
-L +5V #PWR61
+L +5V #PWR047
 U 1 1 583A2A93
 P 4100 1500
-F 0 "#PWR61" H 4100 1350 50  0001 C CNN
+F 0 "#PWR047" H 4100 1350 50  0001 C CNN
 F 1 "+5V" H 4100 1640 50  0000 C CNN
 F 2 "" H 4100 1500 50  0000 C CNN
@@
 $EndComp
 $Comp
-L GND #PWR60
+L GND #PWR048
 U 1 1 583BF574
 P 4000 1900
-F 0 "#PWR60" H 4000 1650 50  0001 C CNN
+F 0 "#PWR048" H 4000 1650 50  0001 C CNN
 F 1 "GND" H 4000 1750 50  0000 C CNN
 F 2 "" H 4000 1900 50  0000 C CNN
@@
 $EndComp
 $Comp
-L GND #PWR51
+L GND #PWR049
 U 1 1 583BF590
 P 2800 1900
-F 0 "#PWR51" H 2800 1650 50  0001 C CNN
+F 0 "#PWR049" H 2800 1650 50  0001 C CNN
 F 1 "GND" H 2800 1750 50  0000 C CNN
 F 2 "" H 2800 1900 50  0000 C CNN
@@
 $EndComp
 $Comp
-L +3V3 #PWR67
+L +3V3 #PWR050
 U 1 1 583D6746
 P 6400 1700
-F 0 "#PWR67" H 6400 1550 50  0001 C CNN
+F 0 "#PWR050" H 6400 1550 50  0001 C CNN
 F 1 "+3V3" H 6400 1840 50  0000 C CNN
 F 2 "" H 6400 1700 50  0000 C CNN
@@
 $EndComp
 $Comp
-L GND #PWR68
+L GND #PWR051
 U 1 1 583D6797
 P 6400 2400
-F 0 "#PWR68" H 6400 2150 50  0001 C CNN
+F 0 "#PWR051" H 6400 2150 50  0001 C CNN
 F 1 "GND" H 6400 2250 50  0000 C CNN
 F 2 "" H 6400 2400 50  0000 C CNN
@@
 Connection ~ 3700 2500
 $Comp
-L GND #PWR56
+L GND #PWR052
 U 1 1 58410F1B
 P 3700 2900
-F 0 "#PWR56" H 3700 2650 50  0001 C CNN
+F 0 "#PWR052" H 3700 2650 50  0001 C CNN
 F 1 "GND" H 3700 2750 50  0000 C CNN
 F 2 "" H 3700 2900 50  0000 C CNN
@@
 	3700 2900 3700 2800
 $Comp
-L +5V #PWR49
+L +5V #PWR053
 U 1 1 58410FDD
 P 2500 2500
-F 0 "#PWR49" H 2500 2350 50  0001 C CNN
+F 0 "#PWR053" H 2500 2350 50  0001 C CNN
 F 1 "+5V" H 2500 2640 50  0000 C CNN
 F 2 "" H 2500 2500 50  0000 C CNN
@@
 Connection ~ 3900 3500
 $Comp
-L GND #PWR57
+L GND #PWR054
 U 1 1 5841129F
 P 3900 3900
-F 0 "#PWR57" H 3900 3650 50  0001 C CNN
+F 0 "#PWR054" H 3900 3650 50  0001 C CNN
 F 1 "GND" H 3900 3750 50  0000 C CNN
 F 2 "" H 3900 3900 50  0000 C CNN
@@
 	3900 3900 3900 3800
 $Comp
-L GND #PWR53
+L GND #PWR055
 U 1 1 584112A6
 P 3200 4000
-F 0 "#PWR53" H 3200 3750 50  0001 C CNN
+F 0 "#PWR055" H 3200 3750 50  0001 C CNN
 F 1 "GND" H 3200 3850 50  0000 C CNN
 F 2 "" H 3200 4000 50  0000 C CNN
@@
 $EndComp
 $Comp
-L +3V3 #PWR43
+L +3V3 #PWR056
 U 1 1 5841154E
 P 2000 3500
-F 0 "#PWR43" H 2000 3350 50  0001 C CNN
+F 0 "#PWR056" H 2000 3350 50  0001 C CNN
 F 1 "+3V3" H 2000 3640 50  0000 C CNN
 F 2 "" H 2000 3500 50  0000 C CNN
@@
 Connection ~ 3900 4500
 $Comp
-L GND #PWR58
+L GND #PWR057
 U 1 1 58411A77
 P 3900 4900
-F 0 "#PWR58" H 3900 4650 50  0001 C CNN
+F 0 "#PWR057" H 3900 4650 50  0001 C CNN
 F 1 "GND" H 3900 4750 50  0000 C CNN
 F 2 "" H 3900 4900 50  0000 C CNN
@@
 	3900 4900 3900 4800
 $Comp
-L GND #PWR54
+L GND #PWR058
 U 1 1 58411A7E
 P 3200 5000
-F 0 "#PWR54" H 3200 4750 50  0001 C CNN
+F 0 "#PWR058" H 3200 4750 50  0001 C CNN
 F 1 "GND" H 3200 4850 50  0000 C CNN
 F 2 "" H 3200 5000 50  0000 C CNN
@@
 $EndComp
 $Comp
-L +3V3 #PWR44
+L +3V3 #PWR059
 U 1 1 58411A84
 P 2000 4500
-F 0 "#PWR44" H 2000 4350 50  0001 C CNN
+F 0 "#PWR059" H 2000 4350 50  0001 C CNN
 F 1 "+3V3" H 2000 4640 50  0000 C CNN
 F 2 "" H 2000 4500 50  0000 C CNN
@@
 Connection ~ 4700 5500
 $Comp
-L GND #PWR65
+L GND #PWR060
 U 1 1 58411BFE
 P 4700 5900
-F 0 "#PWR65" H 4700 5650 50  0001 C CNN
+F 0 "#PWR060" H 4700 5650 50  0001 C CNN
 F 1 "GND" H 4700 5750 50  0000 C CNN
 F 2 "" H 4700 5900 50  0000 C CNN
@@
 	4700 5900 4700 5800
 $Comp
-L GND #PWR55
+L GND #PWR061
 U 1 1 58411C05
 P 3200 6000
-F 0 "#PWR55" H 3200 5750 50  0001 C CNN
+F 0 "#PWR061" H 3200 5750 50  0001 C CNN
 F 1 "GND" H 3200 5850 50  0000 C CNN
 F 2 "" H 3200 6000 50  0000 C CNN
@@
 $EndComp
 $Comp
-L +3V3 #PWR45
+L +3V3 #PWR062
 U 1 1 58411C0B
 P 2000 5500
-F 0 "#PWR45" H 2000 5350 50  0001 C CNN
+F 0 "#PWR062" H 2000 5350 50  0001 C CNN
 F 1 "+3V3" H 2000 5640 50  0000 C CNN
 F 2 "" H 2000 5500 50  0000 C CNN
@@
 	2700 2800 2700 2900
 $Comp
-L GND #PWR50
+L GND #PWR063
 U 1 1 5841303A
 P 2700 2900
-F 0 "#PWR50" H 2700 2650 50  0001 C CNN
+F 0 "#PWR063" H 2700 2650 50  0001 C CNN
 F 1 "GND" H 2700 2750 50  0000 C CNN
 F 2 "" H 2700 2900 50  0000 C CNN
@@
 	2200 3800 2200 3900
 $Comp
-L GND #PWR46
+L GND #PWR064
 U 1 1 584131CE
 P 2200 3900
-F 0 "#PWR46" H 2200 3650 50  0001 C CNN
+F 0 "#PWR064" H 2200 3650 50  0001 C CNN
 F 1 "GND" H 2200 3750 50  0000 C CNN
 F 2 "" H 2200 3900 50  0000 C CNN
@@
 	2200 4800 2200 4900
 $Comp
-L GND #PWR47
+L GND #PWR065
 U 1 1 5841329B
 P 2200 4900
-F 0 "#PWR47" H 2200 4650 50  0001 C CNN
+F 0 "#PWR065" H 2200 4650 50  0001 C CNN
 F 1 "GND" H 2200 4750 50  0000 C CNN
 F 2 "" H 2200 4900 50  0000 C CNN
@@
 	2200 5800 2200 5900
 $Comp
-L GND #PWR48
+L GND #PWR066
 U 1 1 5841348E
 P 2200 5900
-F 0 "#PWR48" H 2200 5650 50  0001 C CNN
+F 0 "#PWR066" H 2200 5650 50  0001 C CNN
 F 1 "GND" H 2200 5750 50  0000 C CNN
 F 2 "" H 2200 5900 50  0000 C CNN
@@
 	3900 5900 3900 6000
 $Comp
-L GND #PWR59
+L GND #PWR067
 U 1 1 58415615
 P 3900 6000
-F 0 "#PWR59" H 3900 5750 50  0001 C CNN
+F 0 "#PWR067" H 3900 5750 50  0001 C CNN
 F 1 "GND" H 3900 5850 50  0000 C CNN
 F 2 "" H 3900 6000 50  0000 C CNN
@@
 	3200 2800 3200 2900
 $Comp
-L GND #PWR52
+L GND #PWR068
 U 1 1 58419672
 P 3200 2900
-F 0 "#PWR52" H 3200 2650 50  0001 C CNN
+F 0 "#PWR068" H 3200 2650 50  0001 C CNN
 F 1 "GND" H 3200 2750 50  0000 C CNN
 F 2 "" H 3200 2900 50  0000 C CNN
@@
 F 0 "J8" H 4100 1770 50  0000 C CNN
 F 1 "TEST_1P" H 4100 1700 50  0000 C CNN
-F 2 "" H 4300 1500 50  0001 C CNN
+F 2 "Measurement_Points:Measurement_Point_Round-SMD-Pad_Small" H 4300 1500 50  0001 C CNN
 F 3 "" H 4300 1500 50  0001 C CNN
 	1    4100 1500
@@
 F 0 "J7" H 2600 1770 50  0000 C CNN
 F 1 "TEST_1P" H 2600 1700 50  0000 C CNN
-F 2 "" H 2800 1500 50  0001 C CNN
+F 2 "Measurement_Points:Measurement_Point_Round-SMD-Pad_Small" H 2800 1500 50  0001 C CNN
 F 3 "" H 2800 1500 50  0001 C CNN
 	1    2600 1500
@@
 F 0 "J9" H 4100 2770 50  0000 C CNN
 F 1 "TEST_1P" H 4100 2700 50  0000 C CNN
-F 2 "" H 4300 2500 50  0001 C CNN
+F 2 "Measurement_Points:Measurement_Point_Round-SMD-Pad_Small" H 4300 2500 50  0001 C CNN
 F 3 "" H 4300 2500 50  0001 C CNN
 	1    4100 2500
@@
 F 0 "J10" H 4300 3770 50  0000 C CNN
 F 1 "TEST_1P" H 4300 3700 50  0000 C CNN
-F 2 "" H 4500 3500 50  0001 C CNN
+F 2 "Measurement_Points:Measurement_Point_Round-SMD-Pad_Small" H 4500 3500 50  0001 C CNN
 F 3 "" H 4500 3500 50  0001 C CNN
 	1    4300 3500
@@
 F 0 "J12" H 5100 5770 50  0000 C CNN
 F 1 "TEST_1P" H 5100 5700 50  0000 C CNN
-F 2 "" H 5300 5500 50  0001 C CNN
+F 2 "Measurement_Points:Measurement_Point_Round-SMD-Pad_Small" H 5300 5500 50  0001 C CNN
 F 3 "" H 5300 5500 50  0001 C CNN
 	1    5100 5500
@@
 F 0 "J11" H 4300 4770 50  0000 C CNN
 F 1 "TEST_1P" H 4300 4700 50  0000 C CNN
-F 2 "" H 4500 4500 50  0001 C CNN
+F 2 "Measurement_Points:Measurement_Point_Round-SMD-Pad_Small" H 4500 4500 50  0001 C CNN
 F 3 "" H 4500 4500 50  0001 C CNN
 	1    4300 4500
@@
 F 0 "J13" H 6400 3770 50  0000 C CNN
 F 1 "TEST_1P" H 6400 3700 50  0000 C CNN
-F 2 "" H 6600 3500 50  0001 C CNN
+F 2 "Pin_Headers:Pin_Header_Straight_1x01_Pitch2.54mm" H 6600 3500 50  0001 C CNN
 F 3 "" H 6600 3500 50  0001 C CNN
 	1    6400 3500
@@
 $EndComp
 $Comp
-L GND #PWR69
+L GND #PWR069
 U 1 1 5A0E8561
 P 6400 3500
-F 0 "#PWR69" H 6400 3250 50  0001 C CNN
+F 0 "#PWR069" H 6400 3250 50  0001 C CNN
 F 1 "GND" H 6400 3350 50  0000 C CNN
 F 2 "" H 6400 3500 50  0000 C CNN
