File: HDMI-to-LH550WF1/LCD-Panel.sch (KiCad schematic (older format))
At the start: 15 parts, among them P3 LH550WF1, U3 TPS65132A0YFF, U4 TPS61161

Commit message: Added test points to LCD-Panel and Power sheets
Parts:
- added J3, J4, J5, J6: TEST_1P, symbol TEST_1P
Connections:
- net LED_A: now also J4.1
- net LED_PWM: now also J3.1
- net VSN: now also J6.1
- net VSP: now also J5.1

Commit message: Assigned test point footprints
Parts:
- J3, J4, J5, J6: footprint (none) -> Measurement_Points:Measurement_Point_Round-SMD-Pad_Small
Changed lines of the file:
@@
 RESET
 $Comp
-L GND #PWR41
+L GND #PWR028
 U 1 1 58392710
 P 8800 4300
-F 0 "#PWR41" H 8800 4050 50  0001 C CNN
+F 0 "#PWR028" H 8800 4050 50  0001 C CNN
 F 1 "GND" H 8800 4150 50  0000 C CNN
 F 2 "" H 8800 4300 50  0000 C CNN
@@
 $EndComp
 $Comp
-L GND #PWR40
+L GND #PWR029
 U 1 1 58392726
 P 7100 4300
-F 0 "#PWR40" H 7100 4050 50  0001 C CNN
+F 0 "#PWR029" H 7100 4050 50  0001 C CNN
 F 1 "GND" H 7100 4150 50  0000 C CNN
 F 2 "" H 7100 4300 50  0000 C CNN
@@
 NoConn ~ 8700 4200
 $Comp
-L +1V8 #PWR42
+L +1V8 #PWR030
 U 1 1 58393DDA
 P 9000 3200
-F 0 "#PWR42" H 9000 3050 50  0001 C CNN
+F 0 "#PWR030" H 9000 3050 50  0001 C CNN
 F 1 "+1V8" H 9000 3340 50  0000 C CNN
 F 2 "" H 9000 3200 50  0000 C CNN
@@
 LED_PWM
 $Comp
-L +5V #PWR33
+L +5V #PWR031
 U 1 1 58394FDE
 P 2600 4500
-F 0 "#PWR33" H 2600 4350 50  0001 C CNN
+F 0 "#PWR031" H 2600 4350 50  0001 C CNN
 F 1 "+5V" H 2600 4640 50  0000 C CNN
 F 2 "" H 2600 4500 50  0000 C CNN
@@
 $EndComp
 $Comp
-L GND #PWR30
+L GND #PWR032
 U 1 1 58395360
 P 2300 4900
-F 0 "#PWR30" H 2300 4650 50  0001 C CNN
+F 0 "#PWR032" H 2300 4650 50  0001 C CNN
 F 1 "GND" H 2300 4750 50  0000 C CNN
 F 2 "" H 2300 4900 50  0000 C CNN
@@
 $EndComp
 $Comp
-L GND #PWR31
+L GND #PWR033
 U 1 1 58395A08
 P 2500 5800
-F 0 "#PWR31" H 2500 5550 50  0001 C CNN
+F 0 "#PWR033" H 2500 5550 50  0001 C CNN
 F 1 "GND" H 2500 5650 50  0000 C CNN
 F 2 "" H 2500 5800 50  0000 C CNN
@@
 $EndComp
 $Comp
-L GND #PWR34
+L GND #PWR034
 U 1 1 58395A97
 P 3200 5800
-F 0 "#PWR34" H 3200 5550 50  0001 C CNN
+F 0 "#PWR034" H 3200 5550 50  0001 C CNN
 F 1 "GND" H 3200 5650 50  0000 C CNN
 F 2 "" H 3200 5800 50  0000 C CNN
@@
 $EndComp
 $Comp
-L GND #PWR35
+L GND #PWR035
 U 1 1 58395AB4
 P 3900 5800
-F 0 "#PWR35" H 3900 5550 50  0001 C CNN
+F 0 "#PWR035" H 3900 5550 50  0001 C CNN
 F 1 "GND" H 3900 5650 50  0000 C CNN
 F 2 "" H 3900 5800 50  0000 C CNN
@@
 $EndComp
 $Comp
-L GND #PWR37
+L GND #PWR036
 U 1 1 583963D4
 P 4200 4900
-F 0 "#PWR37" H 4200 4650 50  0001 C CNN
+F 0 "#PWR036" H 4200 4650 50  0001 C CNN
 F 1 "GND" H 4200 4750 50  0000 C CNN
 F 2 "" H 4200 4900 50  0000 C CNN
@@
 LED_A
 $Comp
-L +5V #PWR28
+L +5V #PWR037
 U 1 1 58397D18
 P 2100 1400
-F 0 "#PWR28" H 2100 1250 50  0001 C CNN
+F 0 "#PWR037" H 2100 1250 50  0001 C CNN
 F 1 "+5V" H 2100 1540 50  0000 C CNN
 F 2 "" H 2100 1400 50  0000 C CNN
@@
 $EndComp
 $Comp
-L GND #PWR29
+L GND #PWR038
 U 1 1 583981F9
 P 2300 1700
-F 0 "#PWR29" H 2300 1450 50  0001 C CNN
+F 0 "#PWR038" H 2300 1450 50  0001 C CNN
 F 1 "GND" H 2300 1550 50  0000 C CNN
 F 2 "" H 2300 1700 50  0000 C CNN
@@
 $EndComp
 $Comp
-L GND #PWR32
+L GND #PWR039
 U 1 1 583983E8
 P 2600 3100
-F 0 "#PWR32" H 2600 2850 50  0001 C CNN
+F 0 "#PWR039" H 2600 2850 50  0001 C CNN
 F 1 "GND" H 2600 2950 50  0000 C CNN
 F 2 "" H 2600 3100 50  0000 C CNN
@@
 $EndComp
 $Comp
-L GND #PWR36
+L GND #PWR040
 U 1 1 58398C7D
 P 4200 2200
-F 0 "#PWR36" H 4200 1950 50  0001 C CNN
+F 0 "#PWR040" H 4200 1950 50  0001 C CNN
 F 1 "GND" H 4200 2050 50  0000 C CNN
 F 2 "" H 4200 2200 50  0000 C CNN
@@
 $EndComp
 $Comp
-L GND #PWR38
+L GND #PWR041
 U 1 1 58398F9F
 P 4500 2200
-F 0 "#PWR38" H 4500 1950 50  0001 C CNN
+F 0 "#PWR041" H 4500 1950 50  0001 C CNN
 F 1 "GND" H 4500 2050 50  0000 C CNN
 F 2 "" H 4500 2200 50  0000 C CNN
@@
 $EndComp
 $Comp
-L GND #PWR39
+L GND #PWR042
 U 1 1 58399019
 P 4500 2800
-F 0 "#PWR39" H 4500 2550 50  0001 C CNN
+F 0 "#PWR042" H 4500 2550 50  0001 C CNN
 F 1 "GND" H 4500 2650 50  0000 C CNN
 F 2 "" H 4500 2800 50  0000 C CNN
@@
 F 0 "J5" H 4900 2170 50  0000 C CNN
 F 1 "TEST_1P" H 4900 2100 50  0000 C CNN
-F 2 "" H 5100 1900 50  0001 C CNN
+F 2 "Measurement_Points:Measurement_Point_Round-SMD-Pad_Small" H 5100 1900 50  0001 C CNN
 F 3 "" H 5100 1900 50  0001 C CNN
 	1    4900 1900
@@
 F 0 "J6" H 4900 2770 50  0000 C CNN
 F 1 "TEST_1P" H 4900 2700 50  0000 C CNN
-F 2 "" H 5100 2500 50  0001 C CNN
+F 2 "Measurement_Points:Measurement_Point_Round-SMD-Pad_Small" H 5100 2500 50  0001 C CNN
 F 3 "" H 5100 2500 50  0001 C CNN
 	1    4900 2500
@@
 F 0 "J4" H 4600 4970 50  0000 C CNN
 F 1 "TEST_1P" H 4600 4900 50  0000 C CNN
-F 2 "" H 4800 4700 50  0001 C CNN
+F 2 "Measurement_Points:Measurement_Point_Round-SMD-Pad_Small" H 4800 4700 50  0001 C CNN
 F 3 "" H 4800 4700 50  0001 C CNN
 	1    4600 4700
@@
 F 0 "J3" H 2100 5570 50  0000 C CNN
 F 1 "TEST_1P" H 2100 5500 50  0000 C CNN
-F 2 "" H 2300 5300 50  0001 C CNN
+F 2 "Measurement_Points:Measurement_Point_Round-SMD-Pad_Small" H 2300 5300 50  0001 C CNN
 F 3 "" H 2300 5300 50  0001 C CNN
 	1    2100 5300
